File: hardware/chubby hat/src/chubby hat.kicad_pcb (KiCad board)
At the start: 2 copper layers, 143.5 x 91.4 mm, 84 parts, among them J1 HUB75, J10 Conn_01x02, J11 Conn_01x04, J12 USB_C_Receptacle_USB2.0, J13 Conn_ARM_JTAG_SWD_10, J14 SWD, J15 5V, J16 5V, J17 5V, J18 5V, J19 5V, J2 HUB75, J20 Conn_ARM_JTAG_SWD_10, J21 TC2030, J3 HUB75, J4 HUB75, J5 HUB75, J6 HUB75, J7 HUB75, J8 HUB75, J9 Screw_Terminal_01x02, Q1 AO3401A, SW2 reset, SW3 boot0, U1 FT2232D, U2 USBLC6-2SC6, U3 STM32F103C8Tx, U4 AMS1117-3.3, Y1 6MHz, Y2 8MHz

Commit message: fixed wrong JTAG signal assignment on FTDI
Connections:
- U1 pad 21: /JTAG.TDI -> /JTAG.TMS
- U1 pad 23: /JTAG.TMS -> /JTAG.TDI
Changed lines of the file:
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@@
       (net 13 "/JTAG.TCK") (pinfunction "ADBUS0"))
     (pad "23" smd roundrect (at 2.25 -4.1625 90) (size 0.3 1.475) (layers "B.Cu" "B.Paste" "B.Mask") (roundrect_rratio 0.25)
-      (net 12 "/JTAG.TMS") (pinfunction "ADBUS1"))
+      (net 11 "/JTAG.TDI") (pinfunction "ADBUS1"))
     (pad "22" smd roundrect (at 1.75 -4.1625 90) (size 0.3 1.475) (layers "B.Cu" "B.Paste" "B.Mask") (roundrect_rratio 0.25)
       (net 6 "/JTAG.TDO") (pinfunction "ADBUS2"))
     (pad "21" smd roundrect (at 1.25 -4.1625 90) (size 0.3 1.475) (layers "B.Cu" "B.Paste" "B.Mask") (roundrect_rratio 0.25)
-      (net 11 "/JTAG.TDI") (pinfunction "ADBUS3"))
+      (net 12 "/JTAG.TMS") (pinfunction "ADBUS3"))
     (pad "20" smd roundrect (at 0.75 -4.1625 90) (size 0.3 1.475) (layers "B.Cu" "B.Paste" "B.Mask") (roundrect_rratio 0.25)
       (net 89 "/FTDI/ADBUS4") (pinfunction "ADBUS4"))
