File: source/template/template.kicad_pcb (KiCad board)
At the start: 2 copper layers, 0 parts

Commit message: make OSH Park 2 layer default
Other:
- rule pad_to_mask_clearance: 0.05 -> 0
- rule solder_mask_min_width: 0.2 -> 0.1016
Changed lines of the file:
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@@
       (dielectric_constraints no)
     )
-    (pad_to_mask_clearance 0.05)
-    (solder_mask_min_width 0.2)
+    (pad_to_mask_clearance 0)
+    (solder_mask_min_width 0.1016)
     (pcbplotparams
       (layerselection 0x00010fc_ffffffff)
